File: pcb/rev.A/zx-supersound.kicad_pcb (KiCad board)
At the start: 2 copper layers, 170 x 63.6 mm, 195 parts, among them J1 PJ307, J2 PinHeader, J3 Conn_01x04, J4 Conn_02x31_Row_Letter_First, J6 Conn_02x03_Odd_Even, SW1 SW_DIP_x05, SW2 SW_DIP_x05, U1 MCP602, U10 YM3014B, U11 SAM2695, U12 AS6C4008-55SIN, U13 AMS1117-3.3, U14 SAA1099, U15 8580, U16 AMS1117-3.3, U18 AMS1117-ADJ, U19 ATmega88PA-AU, U2 MCP602, U3 Z84C0020PEC, U4 YM2203, U5 YM3014B, U6 MCP602, U7 EPM3256ATC144, U8 27C512, U9 YM2203, X1 32MHz

Commit message: wip pcb rev.A
Parts:
- removed C91, C94: 100n, Capacitor_SMD:C_0805_2012Metric_Pad1.18x1.45mm_HandSolder
- removed C93: 10u, Capacitor_SMD:C_0805_2012Metric_Pad1.18x1.45mm_HandSolder
- removed JP9: Jumper_3_Open, Connector_PinHeader_2.54mm:PinHeader_1x03_P2.54mm_Vertical
- removed L1: 27uH, Inductor_SMD:L_6.3x6.3_H3
- removed R67: 240, Resistor_SMD:R_0805_2012Metric_Pad1.20x1.40mm_HandSolder
- removed R69: 1k, Resistor_SMD:R_0805_2012Metric_Pad1.20x1.40mm_HandSolder
- added C92: 10u, Capacitor_SMD:C_1206_3216Metric_Pad1.33x1.80mm_HandSolder, F.Cu at (80.8, 65.9)
- added C96: 10u, Capacitor_SMD:C_1206_3216Metric_Pad1.33x1.80mm_HandSolder, F.Cu at (95.9, 34.4)
- added C98: 10u, Capacitor_SMD:C_1206_3216Metric_Pad1.33x1.80mm_HandSolder, F.Cu at (95.8, 45.5)
- added JP1: Jumper_3_Open, Connector_PinHeader_2.54mm:PinHeader_1x03_P2.54mm_Vertical, F.Cu at (121.8, 59.4)
- added U17: NCP1117-5.0_TO252, Package_TO_SOT_SMD:TO-252-2, F.Cu at (89.0, 34.4)
- added U20: NCP1117-5.0_TO252, Package_TO_SOT_SMD:TO-252-2, F.Cu at (89.0, 45.5)
- added U21: NCP1117-5.0_TO252, Package_TO_SOT_SMD:TO-252-2, F.Cu at (73.9, 65.9)
- added U22: AS6C4008-55SIN, Package_SO:SSOP-32_11.305x20.495mm_P1.27mm, F.Cu at (216.8, 107.6)
- added U23: 74HC245, Package_SO:SOIC-20W_7.5x12.8mm_P1.27mm, F.Cu at (181.7, 71.1)
- C34: footprint Capacitor_THT:CP_Radial_D6.3mm_P2.50mm -> Capacitor_SMD:CP_Elec_6.3x7.7
- C35: value 100n -> 10u; footprint Capacitor_SMD:C_0805_2012Metric_Pad1.18x1.45mm_HandSolder -> Capacitor_SMD:C_1206_3216Metric_Pad1.33x1.80mm_HandSolder
- C36: value 100u -> 10u; footprint Capacitor_THT:CP_Radial_D6.3mm_P2.50mm -> Capacitor_SMD:C_1206_3216Metric_Pad1.33x1.80mm_HandSolder; moved to B.Cu
- C37: value 220u -> 10u; footprint Capacitor_THT:CP_Radial_D10.0mm_P5.00mm -> Capacitor_SMD:C_1206_3216Metric_Pad1.33x1.80mm_HandSolder
- C77, C78: value 10u -> 47u/16V; footprint Capacitor_SMD:CP_Elec_4x5.4 -> Capacitor_Tantalum_SMD:CP_EIA-6032-28_Kemet-C_Pad2.25x2.35mm_HandSolder
- C84: value 47u/16V -> 100u; footprint Capacitor_Tantalum_SMD:CP_EIA-6032-28_Kemet-C_Pad2.25x2.35mm_HandSolder -> Capacitor_SMD:CP_Elec_6.3x7.7
- C86, C87, C88, C89, R23, R40: moved to B.Cu
- C90: value 100n -> 47u/16V; footprint Capacitor_SMD:C_0805_2012Metric_Pad1.18x1.45mm_HandSolder -> Capacitor_Tantalum_SMD:CP_EIA-6032-28_Kemet-C_Pad2.25x2.35mm_HandSolder
- LOGO1: footprint my:black-mage2 -> mygraphic:black-mage-9.6x6.5
- R15, R25: moved to F.Cu
- U1, U2, U6: footprint Package_DIP:DIP-8_W7.62mm_Socket -> Package_SO:SOIC-8_3.9x4.9mm_P1.27mm
- U18: value AMS1117-ADJ -> L78L09_SOT89; footprint Package_TO_SOT_SMD:SOT-223-3_TabPin2 -> Package_TO_SOT_SMD:SOT-89-3
- X1: footprint Oscillator:Oscillator_SMD_EuroQuartz_XO91-4Pin_7.0x5.0mm_HandSoldering -> Oscillator:Oscillator_SMD_SeikoEpson_SG8002CA-4Pin_7.0x5.0mm
- moved C77 180.1 mm to (66.3, 65.9), turned to 90 degrees
- moved C78 168.1 mm to (81.4, 34.4), turned to -90 degrees
- moved C79 133.4 mm to (116.4, 41.8)
- moved R53 133.1 mm to (124.1, 44.1)
- moved C72 133.1 mm to (121.8, 44.1)
- moved R54 133.1 mm to (126.7, 44.1)
- moved JP6 133.0 mm to (139.1, 59.4)
- moved JP7 133.0 mm to (130.4, 59.4)
- moved R55 133.0 mm to (134.1, 53.2)
- moved U15 133.0 mm to (121.6, 56.0)
- moved J6 133.0 mm to (133.2, 46.9)
- moved R68 133.0 mm to (138.2, 53.2)
- moved C73 132.9 mm to (124.1, 52.6)
- moved C74 132.9 mm to (126.4, 52.6)
- moved C75 132.9 mm to (128.6, 52.6)
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Connections:
- C12 pad 2: GND -> GNDA
- C15 pad 2: GND -> GNDA
- C16 pad 2: GND -> GNDA
- C17 pad 2: GND -> GNDA
- C20 pad 2: GND -> GNDA
- C23 pad 2: GND -> GNDA
- C24 pad 2: GND -> GNDA
- C25 pad 2: GND -> GNDA
- C26 pad 2: GND -> GNDA
- C27 pad 2: GND -> GNDA
- C28 pad 2: GND -> GNDA
- C29 pad 2: GND -> GNDA
- C30 pad 2: GND -> GNDA
- C31 pad 2: GND -> GNDA
- C32 pad 2: GND -> GNDA
- C33 pad 2: GND -> GNDA
- C35 pad 1: GND -> +5V
- C35 pad 2: +5V -> GND
- C37 pad 1: +5VA -> +12V
- C37 pad 2: GND -> GNDA
- C41 pad 1: GND -> GNDA
- C42 pad 1: +5V -> +12V
- C42 pad 2: GND -> GNDA
- C43 pad 2: GND -> GNDA
- C44 pad 2: GND -> GNDA
- C45 pad 2: GND -> GNDA
- C46 pad 2: GND -> GNDA
- C47 pad 2: GND -> GNDA
- C6 pad 1: GND -> GNDA
- C60 pad 1: GND -> GNDA
- C60 pad 2: +5VA -> +5VA_1
- C61 pad 1: GND -> GNDA
- C61 pad 2: +5VA -> +5VA_2
- C62 pad 1: GND -> GNDA
- C62 pad 2: +5VA -> +5VA_1
- C63 pad 1: GND -> GNDA
- C63 pad 2: +5VA -> +5VA_2
- C64 pad 1: GND -> GNDA
- C64 pad 2: +5VA -> +5VA_2
- C65 pad 1: GND -> GNDA
- C66 pad 1: GND -> GNDA
- C67 pad 1: GND -> GNDA
- C68 pad 2: GND -> GNDA
- C69 pad 2: GND -> GNDA
- C70 pad 2: GND -> GNDA
- C71 pad 2: GND -> GNDA
- C77 pad 1: Net-(C77-Pad1) -> +5VA
- C77 pad 2: Net-(C77-Pad2) -> GNDA
- C78 pad 1: Net-(C78-Pad1) -> +5VA_1
- C78 pad 2: Net-(C78-Pad2) -> GNDA
- C79 pad 1: Net-(C77-Pad1) -> Net-(C79-Pad1)
- C80 pad 1: Net-(C78-Pad1) -> Net-(C80-Pad1)
- C82 pad 1: Net-(C78-Pad1) -> Net-(C80-Pad1)
- C82 pad 2: Net-(C82-Pad2) -> Net-(R66-Pad2)
- C83 pad 2: GND -> GNDA
- C84 pad 1: +5V -> +12V
- C85 pad 2: GND -> GNDA
- C86 pad 2: GND -> GNDA
- C87 pad 1: +5V -> GND
- C87 pad 2: GND -> +5V
- C88 pad 1: +3V3 -> GND
- C88 pad 2: GND -> +5V
- C89 pad 1: +3V3 -> GNDA
- C89 pad 2: GND -> +5VA_1
- C90 pad 1: +3V3 -> +5VA_2
- C90 pad 2: GND -> GNDA
- R10 pad 1: GND -> GNDA
- R11 pad 1: GND -> GNDA
- R12 pad 1: GND -> GNDA
- R36 pad 1: GND -> GNDA
- R37 pad 1: GND -> GNDA
- R38 pad 1: GND -> GNDA
- R53 pad 1: Net-(C77-Pad1) -> Net-(C79-Pad1)
- R58 pad 2: Net-(C77-Pad2) -> Net-(C79-Pad2)
- R60 pad 1: Net-(C78-Pad1) -> Net-(C80-Pad1)
- R61 pad 2: Net-(C82-Pad2) -> Net-(R66-Pad2)
- R63 pad 1: Net-(C78-Pad1) -> Net-(C80-Pad1)
- R66 pad 2: Net-(C78-Pad2) -> Net-(R66-Pad2)
- R9 pad 2: GND -> GNDA
- U1 pad 4: GND -> GNDA
- U10 pad 1: +5VA -> +5VA_2
- U10 pad 6: GND -> GNDA
- U11 pad 10: GND -> GNDA
- U11 pad 13: GND -> GNDA
- U11 pad 14: GND -> GNDA
- U11 pad 15: GND -> GNDA
- U11 pad 18: GND -> GNDA
- U11 pad 25: GND -> GNDA
- U11 pad 36: GND -> GNDA
- U11 pad 4: GND -> GNDA
- U11 pad 45: GND -> GNDA
- U11 pad 48: GND -> GNDA
- U11 pad 49: GND -> GNDA
- U11 pad 7: GND -> GNDA
- U11 pad 9: GND -> GNDA
- U14 pad 18: +5VA -> +5VA_2
- U14 pad 9: GND -> GNDA
- U15 pad 27: Net-(C77-Pad1) -> Net-(C79-Pad1)
- U16 pad 1: GND -> GNDA
- U16 pad 3: +5V -> +12V
- U18 pad 1: Net-(R67-Pad1) -> +9V
- U18 pad 2: +6V -> GNDA
- U18 pad 3: VDDA -> +12V
- U2 pad 4: GND -> GNDA
- U4 pad 1: GND -> GNDA
- U4 pad 17: GND -> GNDA
- U4 pad 21: +5VA -> +5VA_1
- U5 pad 1: +5VA -> +5VA_1
- U5 pad 6: GND -> GNDA
- U6 pad 4: GND -> GNDA
- U9 pad 1: GND -> GNDA
- U9 pad 17: GND -> GNDA
- U9 pad 21: +5VA -> +5VA_2
- X1 pad 1: +3V3 -> +5V
- X1 pad 4: +3V3 -> +5V
Other:
- board text added: "•Turbo Sound FM• •General Sound• •SAA1099• •MIDI•"

Commit message: wip pcb rev.A
Parts:
- removed C37: 10u, Capacitor_SMD:C_1206_3216Metric_Pad1.33x1.80mm_HandSolder
- removed C41, C72, C85, C86: 100n, Capacitor_SMD:C_0805_2012Metric_Pad1.18x1.45mm_HandSolder
- removed C73, C75: 470p, Capacitor_SMD:C_0805_2012Metric_Pad1.18x1.45mm_HandSolder
- removed C74, C76: 22n, Capacitor_SMD:C_0805_2012Metric_Pad1.18x1.45mm_HandSolder
- removed C79, C82: 10u, Capacitor_SMD:CP_Elec_4x5.4
- removed C80: 1n, Capacitor_SMD:C_0805_2012Metric_Pad1.18x1.45mm_HandSolder
- removed C81: 47u/16V, Capacitor_Tantalum_SMD:CP_EIA-6032-28_Kemet-C_Pad2.25x2.35mm_HandSolder
- removed J6: Conn_02x03_Odd_Even, Connector_PinHeader_2.54mm:PinHeader_2x03_P2.54mm_Vertical
- removed JP1, JP5, JP6, JP7: Jumper_3_Open, Connector_PinHeader_2.54mm:PinHeader_1x03_P2.54mm_Vertical
- removed JP8: Jumper, Connector_PinHeader_2.54mm:PinHeader_1x02_P2.54mm_Vertical
- removed R55, R56: 10k, Resistor_SMD:R_0805_2012Metric_Pad1.20x1.40mm_HandSolder
- removed R57, R58, R61, R66: 22k, Resistor_SMD:R_0805_2012Metric_Pad1.20x1.40mm_HandSolder
- removed R60: 4.7k, Resistor_SMD:R_0805_2012Metric_Pad1.20x1.40mm_HandSolder
- removed R62, R68: 1k, Resistor_SMD:R_0805_2012Metric_Pad1.20x1.40mm_HandSolder
- removed R63: 2.2k, Resistor_SMD:R_0805_2012Metric_Pad1.20x1.40mm_HandSolder
- removed R65: 240k, Resistor_SMD:R_0805_2012Metric_Pad1.20x1.40mm_HandSolder
- removed SW1: SW_DIP_x05, Button_Switch_THT:SW_DIP_SPSTx05_Slide_6.7x14.26mm_W7.62mm_P2.54mm_LowProfile
- removed U15: 8580, Package_DIP:DIP-28_W15.24mm_Socket
- removed U18: L78L09_SOT89, Package_TO_SOT_SMD:SOT-89-3
- removed U19: ATmega88PA-AU, Package_QFP:TQFP-32_7x7mm_P0.8mm
- C42, C83, C92, C96, C98: moved to B.Cu
- R53: value 1k -> 10k; moved to B.Cu
- R54: value 330k -> 10k; moved to B.Cu
- moved R53 81.6 mm to (202.4, 67.2)
- moved R54 76.7 mm to (199.8, 67.2)
- moved C77 49.3 mm to (80.2, 113.2), turned to -90 degrees
- moved C92 49.2 mm to (68.8, 113.6), turned to 90 degrees
- moved U21 47.7 mm to (71.8, 113.6), turned to 0 degrees
- moved C96 40.5 mm to (70.8, 66.1), turned to 90 degrees
- moved U17 34.7 mm to (75.0, 66.1), turned to 0 degrees
- moved C78 31.7 mm to (83.2, 66.1), turned to 90 degrees
- moved C90 28.6 mm to (101.2, 66.1), turned to 90 degrees
- moved C98 21.8 mm to (88.8, 66.1), turned to 90 degrees
- moved U20 21.0 mm to (93.1, 66.1), turned to 0 degrees
- moved R20 14.8 mm to (73.9, 94.0)
- moved R7 10.4 mm to (71.7, 94.0)
- moved C83 9.90 mm to (102.9, 113.6), turned to 0 degrees
- moved C15 8.95 mm to (85.8, 73.6)
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Connections:
- net CLK32 renamed /CLK32
- C12 pad 2: GNDA -> GND
- C15 pad 2: GNDA -> GND
- C16 pad 2: GNDA -> GND
- C17 pad 2: GNDA -> GND
- C20 pad 2: GNDA -> GND
- C23 pad 2: GNDA -> GND
- C24 pad 2: GNDA -> GND
- C25 pad 2: GNDA -> GND
- C26 pad 2: GNDA -> GND
- C27 pad 2: GNDA -> GND
- C28 pad 2: GNDA -> GND
- C29 pad 2: GNDA -> GND
- C30 pad 2: GNDA -> GND
- C31 pad 2: GNDA -> GND
- C32 pad 2: GNDA -> GND
- C33 pad 2: GNDA -> GND
- C42 pad 2: GNDA -> GND
- C43 pad 2: GNDA -> GND
- C44 pad 2: GNDA -> GND
- C45 pad 2: GNDA -> GND
- C46 pad 2: GNDA -> GND
- C47 pad 2: GNDA -> GND
- C6 pad 1: GNDA -> GND
- C60 pad 1: GNDA -> GND
- C61 pad 1: GNDA -> GND
- C62 pad 1: GNDA -> GND
- C63 pad 1: GNDA -> GND
- C64 pad 1: GNDA -> GND
- C65 pad 1: GNDA -> GND
- C66 pad 1: GNDA -> GND
- C67 pad 1: GNDA -> GND
- C68 pad 2: GNDA -> GND
- C69 pad 2: GNDA -> GND
- C70 pad 2: GNDA -> GND
- C71 pad 2: GNDA -> GND
- C77 pad 2: GNDA -> GND
- C78 pad 2: GNDA -> GND
- C83 pad 2: GNDA -> GND
- C89 pad 1: GNDA -> GND
- C90 pad 2: GNDA -> GND
- C92 pad 2: GNDA -> GND
- C96 pad 2: GNDA -> GND
- C98 pad 2: GNDA -> GND
- R10 pad 1: GNDA -> GND
- R11 pad 1: GNDA -> GND
- R12 pad 1: GNDA -> GND
- R26 pad 2: /GDAC0 -> Net-(R26-Pad2)
- R32 pad 2: /GDAC1 -> Net-(R32-Pad2)
- R35 pad 2: /GDAC2 -> Net-(R35-Pad2)
- R36 pad 1: GNDA -> GND
- R37 pad 1: GNDA -> GND
- R38 pad 1: GNDA -> GND
- R39 pad 2: /GDAC3 -> Net-(R39-Pad2)
- R49 pad 2: /CFG2 -> /CFG0
- R51 pad 2: /CFG0 -> /CFG2
- R53 pad 1: Net-(C79-Pad1) -> +5V
- R53 pad 2: GND -> /CFG4
- R54 pad 1: Net-(R54-Pad1) -> +5V
- R54 pad 2: GND -> /CFG3
- R9 pad 2: GNDA -> GND
- SW2 pad 1: unconnected-(SW2-Pad1) -> /CFG0
- SW2 pad 10: unconnected-(SW2-Pad10) -> GND
- SW2 pad 2: unconnected-(SW2-Pad2) -> /CFG1
- SW2 pad 3: unconnected-(SW2-Pad3) -> /CFG2
- SW2 pad 4: unconnected-(SW2-Pad4) -> /CFG3
- SW2 pad 5: unconnected-(SW2-Pad5) -> /CFG4
- SW2 pad 6: unconnected-(SW2-Pad6) -> GND
- SW2 pad 7: unconnected-(SW2-Pad7) -> GND
- SW2 pad 8: unconnected-(SW2-Pad8) -> GND
- SW2 pad 9: unconnected-(SW2-Pad9) -> GND
- U1 pad 4: GNDA -> GND
- U10 pad 6: GNDA -> GND
- U11 pad 10: GNDA -> GND
- U11 pad 13: GNDA -> GND
- U11 pad 14: GNDA -> GND
- U11 pad 15: GNDA -> GND
- U11 pad 18: GNDA -> GND
- U11 pad 25: GNDA -> GND
- U11 pad 36: GNDA -> GND
- U11 pad 4: GNDA -> GND
- U11 pad 45: GNDA -> GND
- U11 pad 48: GNDA -> GND
- U11 pad 49: GNDA -> GND
- U11 pad 7: GNDA -> GND
- U11 pad 9: GNDA -> GND
- U12 pad 13: /GD0 -> /GD5
- U12 pad 14: /GD1 -> /GD3
- U12 pad 15: /GD2 -> /GD1
- U12 pad 17: /GD3 -> /GD0
- U12 pad 18: /GD4 -> /GD2
- U12 pad 19: /GD5 -> /GD4
- U12 pad 22: /~{GRAM} -> /~{GRAM1}
- U12 pad 28: /GA13 -> /GA14
- U12 pad 3: /GA14 -> /GA7
- U12 pad 5: /GA7 -> /GA13
- U14 pad 9: GNDA -> GND
- U16 pad 1: GNDA -> GND
- U17 pad 1: GNDA -> GND
- U2 pad 4: GNDA -> GND
- U20 pad 1: GNDA -> GND
- U21 pad 1: GNDA -> GND
- U22 pad 13: /GD0 -> /GD5
- U22 pad 14: /GD1 -> /GD3
- U22 pad 15: /GD2 -> /GD1
- U22 pad 17: /GD3 -> /GD0
- U22 pad 18: /GD4 -> /GD2
- U22 pad 19: /GD5 -> /GD4
- U22 pad 28: /GA13 -> /GA14
- U22 pad 3: /GA14 -> /GA7
- U22 pad 5: /GA7 -> /GA13
- U23 pad 10: GNDA -> GND
- U23 pad 11: unconnected-(U23-Pad11) -> Net-(R26-Pad2)
- U23 pad 13: unconnected-(U23-Pad13) -> Net-(R32-Pad2)
- U23 pad 15: unconnected-(U23-Pad15) -> Net-(R35-Pad2)
- U23 pad 17: unconnected-(U23-Pad17) -> Net-(R39-Pad2)
- U23 pad 19: GNDA -> GND
- U23 pad 3: /GDAC0 -> /GDAC3
- U23 pad 5: /GDAC1 -> /GDAC2
- U23 pad 7: /GDAC2 -> /GDAC1
- U23 pad 9: /GDAC3 -> /GDAC0
- U4 pad 1: GNDA -> GND
- U4 pad 17: GNDA -> GND
- U5 pad 6: GNDA -> GND
- U6 pad 4: GNDA -> GND
- U7 pad 1: /~{NMI} -> A8
- U7 pad 10: /AD4 -> /GA13
- U7 pad 100: A12 -> /AD7
- U7 pad 101: A9 -> /~{SAA_CS}
- U7 pad 102: A11 -> /SAA_CLK
- U7 pad 103: A10 -> /MIDI_CLK
- U7 pad 106: /~{ROMCSB} -> A14
- U7 pad 107: ~{IORQ} -> A15
- U7 pad 108: D7 -> A12
- U7 pad 109: ~{WR} -> A13
- U7 pad 11: /AD5 -> /GA14
- U7 pad 110: D6 -> D7
- U7 pad 111: ~{RD} -> ~{DOS}
- U7 pad 112: D5 -> D0
- U7 pad 113: ~{IORQGE1} -> D1
- U7 pad 116: A13 -> D2
- U7 pad 117: D4 -> A0
- U7 pad 118: D3 -> D6
- U7 pad 119: A15 -> A1
- U7 pad 12: /AD6 -> /GA15
- U7 pad 120: A14 -> D5
- U7 pad 121: ~{M1} -> A2
- U7 pad 122: /~{RFSH} -> D3
- U7 pad 125: /CLKCPU -> unconnected-(U7-Pad125)
- U7 pad 131: /~{MREQ} -> A3
- U7 pad 132: A7 -> D4
- U7 pad 133: A6 -> ~{IORQGE1}
- U7 pad 134: A4 -> ~{IORQ}
- U7 pad 136: A3 -> ~{RD}
- U7 pad 137: A2 -> ~{WR}
- U7 pad 138: A1 -> ~{WAIT}
- U7 pad 139: A0 -> A7
- U7 pad 14: /AD7 -> /GA10
- U7 pad 140: A5 -> A6
- U7 pad 141: D0 -> A4
- U7 pad 142: D1 -> ~{M1}
- U7 pad 143: /~{INT} -> A5
- U7 pad 15: /~{SAA_CS} -> /GA9
- U7 pad 16: /SAA_CLK -> /GA8
- U7 pad 18: /~{YM1_CS} -> /~{GINT}
- U7 pad 19: /~{YM2_CS} -> /GA7
- U7 pad 2: D2 -> A9
- U7 pad 21: /~{AWR} -> /~{GMREQ}
- U7 pad 22: /~{ARD} -> /GA6
- U7 pad 23: /AA0 -> /~{GIORQ}
- U7 pad 25: /YM_M -> /GA5
- U7 pad 27: /AD0 -> /~{GRESET}
- U7 pad 28: /FM2_ENA -> /GA4
- U7 pad 29: /FM1_ENA -> /~{GM1}
- U7 pad 30: /~{RST} -> /GA3
- U7 pad 31: unconnected-(U7-Pad31) -> /GA2
- U7 pad 32: unconnected-(U7-Pad32) -> /GA1
- U7 pad 34: unconnected-(U7-Pad34) -> /GA0
- U7 pad 35: /MIDI_CLK -> /GMA16
- U7 pad 36: /GDAC3 -> /GMA17
- U7 pad 37: /GDAC2 -> /GD0
- U7 pad 38: /GDAC1 -> /GD7
- U7 pad 39: /GDAC0 -> /GD6
- U7 pad 40: /GA11 -> /GD1
- U7 pad 41: /GCLK -> /GD5
- U7 pad 42: /GA12 -> /GD2
- U7 pad 43: /GA13 -> /GD3
- U7 pad 44: /GA14 -> /GD4
- U7 pad 45: /GA15 -> /~{GRD}
- U7 pad 46: /GA10 -> /~{GRAM}
- U7 pad 47: /GA9 -> /~{GWR}
- U7 pad 48: /GA8 -> /GMA18
- U7 pad 49: /~{GINT} -> /GMA15
- U7 pad 5: /BUS1 -> A10
- U7 pad 53: /GA7 -> /~{GROM}
- U7 pad 54: /~{GMREQ} -> /CFG4
- U7 pad 55: /GA6 -> /CFG3
- U7 pad 56: /~{GIORQ} -> /CFG2
- U7 pad 6: /BUS0 -> A11
- U7 pad 60: /GA5 -> /CFG1
- U7 pad 61: /~{GRESET} -> /CFG0
- U7 pad 62: /GA4 -> /GDAC3
- U7 pad 63: /~{GM1} -> /GDAC2
- U7 pad 65: /GA3 -> /GDAC1
- U7 pad 66: /GA2 -> /GDAC0
- U7 pad 67: /GA1 -> unconnected-(U7-Pad67)
- U7 pad 68: /GA0 -> unconnected-(U7-Pad68)
- U7 pad 69: /GMA16 -> unconnected-(U7-Pad69)
- U7 pad 7: /AD1 -> /GA11
- U7 pad 70: /GMA17 -> unconnected-(U7-Pad70)
- U7 pad 71: /GD0 -> unconnected-(U7-Pad71)
- U7 pad 72: /GD7 -> unconnected-(U7-Pad72)
- U7 pad 74: /GD6 -> unconnected-(U7-Pad74)
- U7 pad 75: /GD1 -> unconnected-(U7-Pad75)
- U7 pad 78: /GD5 -> unconnected-(U7-Pad78)
- U7 pad 79: /GD2 -> unconnected-(U7-Pad79)
- U7 pad 8: /AD2 -> /GCLK
- U7 pad 80: /GD3 -> /~{RST}
- U7 pad 81: /GD4 -> /FM2_ENA
- U7 pad 82: /~{GRD} -> /FM1_ENA
- U7 pad 83: /~{GRAM} -> /~{YM1_CS}
- U7 pad 84: /~{GWR} -> /~{YM2_CS}
- U7 pad 86: /GMA18 -> /~{AWR}
- U7 pad 87: /GMA15 -> /~{ARD}
- U7 pad 88: /~{GROM} -> /AA0
- U7 pad 9: /AD3 -> /GA12
- U7 pad 90: /CFG0 -> /YM_M
- U7 pad 91: /CFG1 -> /AD0
- U7 pad 92: /CFG2 -> /AD1
- U7 pad 93: /~{BUSACK} -> /AD2
- U7 pad 96: /~{HALT} -> /AD3
- U7 pad 97: /~{BUSRQ} -> /AD4
- U7 pad 98: A8 -> /AD5
- U7 pad 99: ~{WAIT} -> /AD6
- U9 pad 1: GNDA -> GND
- U9 pad 17: GNDA -> GND
Routing:
- net /AD7: track 0.00 -> 74.4 mm
- net /AD6: track 0.00 -> 71.4 mm
- net /AD5: track 0.00 -> 68.7 mm
- net /AD4: track 0.00 -> 65.9 mm
- net /AD3: track 0.00 -> 63.2 mm
- net /AD2: track 0.00 -> 60.7 mm
- net /AD1: track 0.00 -> 59.2 mm
- net /MIDI_CLK: track 0.00 -> 55.0 mm
- net /GD0: track 0.00 -> 52.8 mm
- net /GD2: track 0.00 -> 48.5 mm
- net /GMA15: track 0.00 -> 48.4 mm, vias 0 -> 2
- net /GA14: track 0.00 -> 43.7 mm
- net /GD4: track 0.00 -> 43.2 mm
- net /GA9: track 0.00 -> 38.5 mm
- net /GA8: track 0.00 -> 38.5 mm
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- added copper zone on B.Cu, net GND

Commit message: wip pcb rev.A
Parts:
- moved C92 43.3 mm to (62.8, 70.7), turned to 0 degrees
- moved U21 40.9 mm to (62.8, 73.7), turned to -90 degrees
- moved C11 37.4 mm to (85.5, 107.2)
- moved C77 35.4 mm to (63.2, 82.1), turned to 180 degrees
- moved C30 33.5 mm to (91.3, 111.3)
- moved C66 33.5 mm to (85.5, 112.6)
- moved U6 33.5 mm to (85.5, 112.6)
- moved C31 33.5 mm to (80.7, 111.7)
- moved R41 33.5 mm to (91.3, 113.7)
- moved C28 33.0 mm to (102.0, 112.0), turned to -90 degrees
- moved C69 31.2 mm to (63.9, 107.9), turned to 90 degrees
- moved R18 30.8 mm to (79.8, 108.3), turned to 0 degrees
- moved C68 30.1 mm to (63.0, 104.9), turned to 0 degrees
- moved C83 29.5 mm to (73.4, 111.9), turned to -90 degrees
- moved C32 28.9 mm to (65.9, 107.9), turned to 90 degrees
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Connections:
- R32 pad 2: Net-(R32-Pad2) -> Net-(U23-Pad14)
- R35 pad 2: Net-(R35-Pad2) -> Net-(U23-Pad16)
- R39 pad 2: Net-(R39-Pad2) -> Net-(U23-Pad18)
- R42 pad 2: +5VA -> +5VA_2
- R43 pad 2: +5VA -> +5VA_2
- R48 pad 2: +5VA -> +5VA_2
- U23 pad 11: Net-(R26-Pad2) -> unconnected-(U23-Pad11)
- U23 pad 12: unconnected-(U23-Pad12) -> Net-(R26-Pad2)
- U23 pad 13: Net-(R32-Pad2) -> unconnected-(U23-Pad13)
- U23 pad 14: unconnected-(U23-Pad14) -> Net-(U23-Pad14)
- U23 pad 15: Net-(R35-Pad2) -> unconnected-(U23-Pad15)
- U23 pad 16: unconnected-(U23-Pad16) -> Net-(U23-Pad16)
- U23 pad 17: Net-(R39-Pad2) -> unconnected-(U23-Pad17)
- U23 pad 18: unconnected-(U23-Pad18) -> Net-(U23-Pad18)
- U23 pad 2: unconnected-(U23-Pad2) -> /GDAC3
- U23 pad 3: /GDAC3 -> unconnected-(U23-Pad3)
- U23 pad 4: unconnected-(U23-Pad4) -> /GDAC2
- U23 pad 5: /GDAC2 -> unconnected-(U23-Pad5)
- U23 pad 6: unconnected-(U23-Pad6) -> /GDAC1
- U23 pad 7: /GDAC1 -> unconnected-(U23-Pad7)
- U23 pad 8: unconnected-(U23-Pad8) -> /GDAC0
- U23 pad 9: /GDAC0 -> unconnected-(U23-Pad9)
- U7 pad 80: /~{RST} -> /FM1_ENA
- U7 pad 81: /FM2_ENA -> /~{YM1_CS}
- U7 pad 82: /FM1_ENA -> /YM_M
- U7 pad 83: /~{YM1_CS} -> /AA0
- U7 pad 84: /~{YM2_CS} -> /~{ARD}
- U7 pad 87: /~{ARD} -> /~{YM2_CS}
- U7 pad 88: /AA0 -> /~{RST}
- U7 pad 90: /YM_M -> /FM2_ENA
Routing:
- net /FM1_ENA: track 0.00 -> 80.5 mm, vias 0 -> 3
- net /FM2_ENA: track 0.00 -> 73.8 mm, vias 0 -> 3
- net Net-(R19-Pad1): track 0.00 -> 69.0 mm
- net Net-(U4-Pad39): track 0.00 -> 67.6 mm, vias 0 -> 1
- net Net-(R1-Pad1): track 0.00 -> 66.8 mm
- net Net-(U10-Pad5): track 0.00 -> 65.5 mm, vias 0 -> 1
- net /~{RST}: track 0.00 -> 63.7 mm, vias 0 -> 4
- net /~{AWR}: track 23.3 -> 63.7 mm, vias 1 -> 4
- net Net-(C23-Pad1): track 0.00 -> 38.3 mm
- net /AA0: track 23.2 -> 61.3 mm, vias 1 -> 4
- net +5VA_2: track 0.00 -> 37.9 mm, vias 0 -> 3
- net GND: track 0.00 -> 33.1 mm, vias 0 -> 23
- net Net-(C16-Pad1): track 0.00 -> 29.8 mm
- net /GDAC0: track 0.00 -> 27.7 mm
- net Net-(C15-Pad1): track 0.00 -> 25.7 mm
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
Commit message: wip pcb rev.A
Parts:
- added J5: Conn_01x04, Connector_PinHeader_2.54mm:PinHeader_1x04_P2.54mm_Vertical, F.Cu at (66.6, 97.8)
- added R55: 24k, Resistor_SMD:R_0805_2012Metric_Pad1.20x1.40mm_HandSolder, F.Cu at (83.4, 97.0)
- added R56: 24k, Resistor_SMD:R_0805_2012Metric_Pad1.20x1.40mm_HandSolder, F.Cu at (83.4, 99.0)
- C83: moved to F.Cu
- moved R2 27.2 mm to (79.2, 101.7), turned to 180 degrees
- moved R33 26.8 mm to (79.2, 105.6), turned to 180 degrees
- moved C71 16.6 mm to (71.2, 114.7), turned to 0 degrees
- moved C68 15.7 mm to (75.6, 114.3), turned to 90 degrees
- moved C69 15.7 mm to (78.6, 113.4), turned to 180 degrees
- moved C42 15.3 mm to (63.1, 103.2), turned to 180 degrees
- moved C43 13.9 mm to (71.2, 112.7), turned to 0 degrees
- moved U16 13.3 mm to (63.1, 102.2)
- moved C32 13.2 mm to (78.6, 111.4), turned to 180 degrees
- moved U11 12.2 mm to (74.8, 111.9), turned to 0 degrees
- moved C26 11.2 mm to (71.2, 110.7), turned to 0 degrees
- moved C33 11.1 mm to (79.1, 109.2), turned to 180 degrees
- moved C83 11.0 mm to (63.1, 108.0), turned to 180 degrees
- moved C31 10.7 mm to (90.9, 108.5), turned to 0 degrees
- moved C70 8.54 mm to (74.7, 109.5), turned to -90 degrees
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Connections:
- net /MIX_L renamed /SND_L
- net /MIX_R renamed /SND_R
- C78 pad 1: +5VA_1 -> +5VA_2
- C90 pad 1: +5VA_2 -> +5VA_1
- R49 pad 1: +5V -> +3V3
- R50 pad 1: +5V -> +3V3
- R51 pad 1: +5V -> +3V3
- R53 pad 1: +5V -> +3V3
- R54 pad 1: +5V -> +3V3
- U17 pad 2: +5VA_1 -> +5VA_2
- U20 pad 2: +5VA_2 -> +5VA_1
- U7 pad 1: A8 -> /~{GRAM2}
- U7 pad 10: /GA13 -> /GA0
- U7 pad 100: /AD7 -> A14
- U7 pad 101: /~{SAA_CS} -> A15
- U7 pad 102: /SAA_CLK -> A12
- U7 pad 103: /MIDI_CLK -> A13
- U7 pad 106: A14 -> D7
- U7 pad 107: A15 -> ~{DOS}
- U7 pad 108: A12 -> D0
- U7 pad 109: A13 -> D1
- U7 pad 11: /GA14 -> /GA1
- U7 pad 110: D7 -> D2
- U7 pad 111: ~{DOS} -> A0
- U7 pad 112: D0 -> D6
- U7 pad 113: D1 -> A1
- U7 pad 116: D2 -> D5
- U7 pad 117: A0 -> A2
- U7 pad 118: D6 -> D3
- U7 pad 119: A1 -> A3
- U7 pad 12: /GA15 -> /GA2
- U7 pad 120: D5 -> D4
- U7 pad 121: A2 -> ~{IORQGE1}
- U7 pad 122: D3 -> ~{IORQ}
- U7 pad 126: unconnected-(U7-Pad126) -> ~{RD}
- U7 pad 131: A3 -> ~{WR}
- U7 pad 132: D4 -> ~{WAIT}
- U7 pad 133: ~{IORQGE1} -> A7
- U7 pad 134: ~{IORQ} -> A6
- U7 pad 136: ~{RD} -> A5
- U7 pad 137: ~{WR} -> ~{M1}
- U7 pad 138: ~{WAIT} -> A4
- U7 pad 139: A7 -> A8
- U7 pad 14: /GA10 -> /GA3
- U7 pad 140: A6 -> A9
- U7 pad 141: A4 -> A10
- U7 pad 142: ~{M1} -> A11
- U7 pad 143: A5 -> unconnected-(U7-Pad143)
- U7 pad 15: /GA9 -> /GA4
- U7 pad 16: /GA8 -> /GA5
- U7 pad 18: /~{GINT} -> /GA6
- U7 pad 2: A9 -> /GMA16
- U7 pad 21: /~{GMREQ} -> /GA8
- U7 pad 22: /GA6 -> /GA9
- U7 pad 23: /~{GIORQ} -> /GA10
- U7 pad 25: /GA5 -> /~{GWR}
- U7 pad 27: /~{GRESET} -> /~{GRD}
- U7 pad 28: /GA4 -> /~{GIORQ}
- U7 pad 29: /~{GM1} -> /~{GMREQ}
- U7 pad 30: /GA3 -> /GA11
- U7 pad 31: /GA2 -> /GA12
- U7 pad 32: /GA1 -> /GA13
- U7 pad 34: /GA0 -> /GA14
- U7 pad 35: /GMA16 -> /GA15
- U7 pad 36: /GMA17 -> /~{GINT}
- U7 pad 37: /GD0 -> /GD3
- U7 pad 38: /GD7 -> /GD5
- U7 pad 40: /GD1 -> /GD4
- U7 pad 41: /GD5 -> /GCLK
- U7 pad 43: /GD3 -> /GD7
- U7 pad 44: /GD4 -> /GD0
- U7 pad 45: /~{GRD} -> /GD1
- U7 pad 46: /~{GRAM} -> /~{GROM}
- U7 pad 47: /~{GWR} -> /GMA15
- U7 pad 48: /GMA18 -> /CFG0
- U7 pad 49: /GMA15 -> /CFG1
- U7 pad 5: A10 -> /GMA17
- U7 pad 53: /~{GROM} -> /CFG2
- U7 pad 54: /CFG4 -> /CFG3
- U7 pad 55: /CFG3 -> /CFG4
- U7 pad 56: /CFG2 -> unconnected-(U7-Pad56)
- U7 pad 6: A11 -> /GMA18
- U7 pad 60: /CFG1 -> /GDAC3
- U7 pad 61: /CFG0 -> /GDAC2
- U7 pad 62: /GDAC3 -> /GDAC1
- U7 pad 63: /GDAC2 -> /GDAC0
- U7 pad 65: /GDAC1 -> unconnected-(U7-Pad65)
- U7 pad 66: /GDAC0 -> unconnected-(U7-Pad66)
- U7 pad 7: /GA11 -> /~{GRAM1}
- U7 pad 74: unconnected-(U7-Pad74) -> /FM1_ENA
- U7 pad 75: unconnected-(U7-Pad75) -> /YM_M
- U7 pad 78: unconnected-(U7-Pad78) -> /AA0
- U7 pad 79: unconnected-(U7-Pad79) -> /~{ARD}
- U7 pad 8: /GCLK -> /~{GM1}
- U7 pad 80: /FM1_ENA -> /~{AWR}
- U7 pad 82: /YM_M -> /~{YM2_CS}
- U7 pad 83: /AA0 -> /~{RST}
- U7 pad 84: /~{ARD} -> /FM2_ENA
- U7 pad 86: /~{AWR} -> /AD0
- U7 pad 87: /~{YM2_CS} -> /AD1
- U7 pad 88: /~{RST} -> /AD2
- U7 pad 9: /GA12 -> /~{GRESET}
- U7 pad 90: /FM2_ENA -> /AD3
- U7 pad 91: /AD0 -> /AD4
- U7 pad 92: /AD1 -> /AD5
- U7 pad 93: /AD2 -> /AD6
- U7 pad 96: /AD3 -> /AD7
- U7 pad 97: /AD4 -> /~{SAA_CS}
- U7 pad 98: /AD5 -> /SAA_CLK
- U7 pad 99: /AD6 -> /MIDI_CLK
Routing:
- net GND: track 33.1 -> 217.8 mm, vias 23 -> 139
- net +3V3: track 0.00 -> 168.1 mm, vias 0 -> 13
- net /MIDI_IN: track 0.00 -> 117.8 mm, vias 0 -> 2
- net /~{RST}: track 63.7 -> 149.0 mm, vias 4 -> 8
- net +3.3VA: track 0.00 -> 73.7 mm, vias 0 -> 12
- net +12V: track 17.9 -> 78.3 mm, vias 0 -> 4
- net /TDO: track 0.00 -> 59.0 mm, vias 0 -> 3
- net /GMA15: track 48.4 -> 104.8 mm, vias 2 -> 3
- net /~{GWR}: track 18.8 -> 68.0 mm, vias 0 -> 4
- net /~{GROM}: track 0.00 -> 48.1 mm, vias 0 -> 2
- net Net-(C21-Pad2): track 3.91 -> 51.7 mm
- net /TCK: track 2.20 -> 49.9 mm, vias 0 -> 3
- net /MIDI_CLK: track 55.0 -> 102.0 mm
- net /GMA17: track 18.8 -> 65.4 mm, vias 0 -> 2
- net /GMA16: track 18.8 -> 64.6 mm, vias 0 -> 2
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- added copper zone on B.Cu, net +5VA
- added copper zone on B.Cu, net +5VA_1
- added copper zone on B.Cu, net +5VA_2
