File: pcb/rev.A/zx-supersound.kicad_sch (KiCad schematic)
At the start: 195 parts, among them J1 PJ307, J2 PinHeader, J3 Conn_01x04, J4 Conn_02x31_Row_Letter_First, J6 Conn_02x03_Odd_Even, SW1 SW_DIP_x05, SW2 SW_DIP_x05, U1 MCP602, U10 YM3014B, U11 SAM2695, U12 AS6C4008-55SIN, U13 AMS1117-3.3, U14 SAA1099, U15 8580, U16 AMS1117-3.3, U18 AMS1117-ADJ, U19 ATmega88PA-AU, U2 MCP602, U3 Z84C0020PEC, U4 YM2203, U5 YM3014B, U6 MCP602, U7 EPM3256ATC144, U8 27C512, U9 YM2203, X1 32MHz

Commit message: wip pcb rev.A
Parts:
- removed C36: 100u, Capacitor_THT:CP_Radial_D6.3mm_P2.50mm, symbol Device:CP
- removed C37: 220u, Capacitor_THT:CP_Radial_D10.0mm_P5.00mm, symbol Device:CP
- removed C90, C91, C94: 100n, Capacitor_SMD:C_0805_2012Metric_Pad1.18x1.45mm_HandSolder, symbol Device:C
- removed C93: 10u, Capacitor_SMD:C_0805_2012Metric_Pad1.18x1.45mm_HandSolder, symbol Device:C
- removed JP9: Jumper_3_Open, Connector_PinHeader_2.54mm:PinHeader_1x03_P2.54mm_Vertical, symbol Jumper:Jumper_3_Open
- removed L1: 27uH, Inductor_SMD:L_6.3x6.3_H3, symbol Device:L
- removed R67: 240, Resistor_SMD:R_0805_2012Metric_Pad1.20x1.40mm_HandSolder, symbol Device:R
- removed R69: 1k, Resistor_SMD:R_0805_2012Metric_Pad1.20x1.40mm_HandSolder, symbol Device:R
- removed U18: AMS1117-ADJ, Package_TO_SOT_SMD:SOT-223-3_TabPin2, symbol Regulator_Linear:AZ1117-ADJ
- added C36, C37, C92, C96, C98: 10u, Capacitor_SMD:C_1206_3216Metric_Pad1.33x1.80mm_HandSolder, symbol Device:C
- added C90: 47u/16V, Capacitor_Tantalum_SMD:CP_EIA-6032-28_Kemet-C_Pad2.25x2.35mm_HandSolder, symbol Device:CP
- added JP1: Jumper_3_Open, Connector_PinHeader_2.54mm:PinHeader_1x03_P2.54mm_Vertical, symbol Jumper:Jumper_3_Open
- added U17, U20, U21: NCP1117-5.0_TO252, Package_TO_SOT_SMD:TO-252-2, symbol Regulator_Linear:NCP1117-5.0_TO252
- added U18: L78L09_SOT89, Package_TO_SOT_SMD:SOT-89-3, symbol Regulator_Linear:L78L09_SOT89
- added U22: AS6C4008-55SIN, Package_SO:SSOP-32_11.305x20.495mm_P1.27mm, symbol my:AS6C4008
- added U23: 74HC245, Package_SO:SOIC-20W_7.5x12.8mm_P1.27mm, symbol 74xx:74HC245
- C34: footprint Capacitor_THT:CP_Radial_D6.3mm_P2.50mm -> Capacitor_SMD:CP_Elec_6.3x7.7
- C35: value 100n -> 10u; footprint Capacitor_SMD:C_0805_2012Metric_Pad1.18x1.45mm_HandSolder -> Capacitor_SMD:C_1206_3216Metric_Pad1.33x1.80mm_HandSolder
- C77, C78: value 10u -> 47u/16V; footprint Capacitor_SMD:CP_Elec_4x5.4 -> Capacitor_Tantalum_SMD:CP_EIA-6032-28_Kemet-C_Pad2.25x2.35mm_HandSolder
- C84: value 47u/16V -> 100u; footprint Capacitor_Tantalum_SMD:CP_EIA-6032-28_Kemet-C_Pad2.25x2.35mm_HandSolder -> Capacitor_SMD:CP_Elec_6.3x7.7
- LOGO1: footprint my:black-mage2 -> mygraphic:black-mage-9.6x6.5
- U1, U2, U6: footprint Package_DIP:DIP-8_W7.62mm_Socket -> Package_SO:SOIC-8_3.9x4.9mm_P1.27mm
- X1: footprint Oscillator:Oscillator_SMD_EuroQuartz_XO91-4Pin_7.0x5.0mm_HandSoldering -> Oscillator:Oscillator_SMD_SeikoEpson_SG8002CA-4Pin_7.0x5.0mm
Connections:
- net +12V: now also C42.1, C84.1, U16.3 (VI), C37.1, C92.1, C96.1, C98.1, JP1.3 (B), U17.3 (VI), U18.3 (IN), U20.3 (VI), U21.3 (VI)
- net +3V3: now also C36.1; no longer C88.1, C89.1, X1.1 (EN), X1.4 (V+)
- net +5V: now also C35.1, C87.2, C88.2, X1.1 (EN), X1.4 (V+), U22.32 (VCC); no longer C35.2, C42.1, C84.1, C87.1, U16.3 (VI)
- net +5VA: now also C77.1, U21.2 (VO); no longer C60.2, C61.2, C62.2, C63.2, C64.2, U10.1 (Vdd), U14.18 (VCC), U4.21 (VDD), U5.1 (Vdd), U9.21 (VDD)
- net +9V: now also JP1.1 (A), U18.1 (OUT)
- net GA0: now also U22.12 (A0)
- net GA1: now also U22.11 (A1)
- net GA10: now also U22.23 (A10)
- net GA11: now also U22.25 (A11)
- net GA12: now also U22.4 (A12)
- net GA13: now also U22.28 (A13)
- net GA14: now also U22.3 (A14)
- net GA2: now also U22.10 (A2)
- net GA3: now also U22.9 (A3)
- net GA4: now also U22.8 (A4)
- net GA5: now also U22.7 (A5)
- net GA6: now also U22.6 (A6)
- net GA7: now also U22.5 (A7)
- net GA8: now also U22.27 (A8)
- net GA9: now also U22.26 (A9)
- net GD0: now also U22.13 (D0)
- net GD1: now also U22.14 (D1)
- net GD2: now also U22.15 (D2)
- net GD3: now also U22.17 (D3)
- net GD4: now also U22.18 (D4)
- net GD5: now also U22.19 (D5)
- net GD6: now also U22.20 (D6)
- net GD7: now also U22.21 (D7)
- net GDAC0: now also U23.3 (A1)
- net GDAC1: now also U23.5 (A3)
- net GDAC2: now also U23.7 (A5)
- net GDAC3: now also U23.9 (A7)
- net GMA15: now also U22.31 (A15)
- net GMA16: now also U22.2 (A16)
- net GMA17: now also U22.1 (A18)
- net GMA18: now also U22.30 (A17)
- net GND: now also C35.2, C87.1, C88.1, C36.2, U22.16 (GND); no longer C12.2, C15.2, C16.2, C17.2, C20.2, C23.2, C24.2, C25.2, C26.2, C27.2, C28.2, C29.2, C30.2, C31.2, C32.2, C33.2, C35.1, C41.1, C42.2, C43.2, C44.2, C45.2, C46.2, C47.2, C6.1, C60.1, C61.1, C62.1, C63.1, C64.1, C65.1, C66.1, C67.1, C68.2, C69.2, C70.2, C71.2, C83.2, C85.2, C86.2, C87.2, C88.2, C89.2, R10.1, R11.1, R12.1, R36.1, R37.1, R38.1, R9.2, U1.4 (V-), U10.6 (Vss), U11.10 (A0), U11.13 (GND), U11.14 (~{CS}), U11.15 (~{RD}), U11.18 (GND), U11.25 (GND), U11.36 (GND), U11.4 (AGND), U11.45 (GND), U11.48 (GND), U11.49 (GND), U11.7 (MICIN), U11.9 (GND), U14.9 (GND), U16.1 (GND), U2.4 (V-), U4.1 (GND), U4.17 (AGND), U5.6 (Vss), U6.4 (V-), U9.1 (GND), U9.17 (AGND)
- net VDDA: now also JP1.2 (C)
- net ~{GRD}: now also U22.24 (~{OE})
- net ~{GWR}: now also U22.29 (~{WE})
- net at R66.2: now also C82.2, R61.2; no longer C78.2
- net at C80.1, C82.1, R60.1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: no longer C78.1
- net at C79.1, R53.1, U15.27 (AUDIO_OUT): no longer C77.1
- net at C79.2, R57.2: now also R58.2
- net GNDA: now reaches C77.2
- net GNDA: now also C12.2, C15.2, C16.2, C17.2, C20.2, C23.2, C24.2, C25.2, C26.2, C27.2, C28.2, C29.2, C30.2, C31.2, C32.2, C33.2, C41.1, C42.2, C43.2, C44.2, C45.2, C46.2, C47.2, C6.1, C60.1, C61.1, C62.1, C63.1, C64.1, C65.1, C66.1, C67.1, C68.2, C69.2, C70.2, C71.2, C78.2, C83.2, C85.2, C86.2, C89.1, R10.1, R11.1, R12.1, R36.1, R37.1, R38.1, R9.2, U1.4 (V-), U10.6 (Vss), U11.10 (A0), U11.13 (GND), U11.14 (~{CS}), U11.15 (~{RD}), U11.18 (GND), U11.25 (GND), U11.36 (GND), U11.4 (AGND), U11.45 (GND), U11.48 (GND), U11.49 (GND), U11.7 (MICIN), U11.9 (GND), U14.9 (GND), U16.1 (GND), U2.4 (V-), U4.1 (GND), U4.17 (AGND), U5.6 (Vss), U6.4 (V-), U9.1 (GND), U9.17 (AGND), C37.2, C90.2, C92.2, C96.2, C98.2, U17.1 (GND), U18.2 (GND), U20.1 (GND), U21.1 (GND), U23.10 (GND), U23.19 (CE); no longer R58.2
- new net +5VA_1: C60.2, C62.2, C78.1, C89.2, U17.2 (VO), U23.1 (A->B), U23.20 (VCC), U4.21 (VDD), U5.1 (Vdd)
- new net +5VA_2: C61.2, C63.2, C64.2, C90.1, U10.1 (Vdd), U14.18 (VCC), U20.2 (VO), U9.21 (VDD)
- new net ~{GRAM2}: U22.22 (~{CE})
Other:
- moved on the sheet: C34, C41, C60, C61, C62, C63, C64, C65, C66, C67, C85, C86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

Commit message: wip pcb rev.A
Parts:
- removed C37: 10u, Capacitor_SMD:C_1206_3216Metric_Pad1.33x1.80mm_HandSolder, symbol Device:C
- removed C41, C72, C85, C86: 100n, Capacitor_SMD:C_0805_2012Metric_Pad1.18x1.45mm_HandSolder, symbol Device:C
- removed C73, C75: 470p, Capacitor_SMD:C_0805_2012Metric_Pad1.18x1.45mm_HandSolder, symbol Device:C
- removed C74, C76: 22n, Capacitor_SMD:C_0805_2012Metric_Pad1.18x1.45mm_HandSolder, symbol Device:C
- removed C79, C82: 10u, Capacitor_SMD:CP_Elec_4x5.4, symbol Device:CP
- removed C80: 1n, Capacitor_SMD:C_0805_2012Metric_Pad1.18x1.45mm_HandSolder, symbol Device:C
- removed C81: 47u/16V, Capacitor_Tantalum_SMD:CP_EIA-6032-28_Kemet-C_Pad2.25x2.35mm_HandSolder, symbol Device:CP
- removed J6: Conn_02x03_Odd_Even, Connector_PinHeader_2.54mm:PinHeader_2x03_P2.54mm_Vertical, symbol Connector_Generic:Conn_02x03_Odd_Even
- removed JP1, JP5, JP6, JP7: Jumper_3_Open, Connector_PinHeader_2.54mm:PinHeader_1x03_P2.54mm_Vertical, symbol Jumper:Jumper_3_Open
- removed JP8: Jumper, Connector_PinHeader_2.54mm:PinHeader_1x02_P2.54mm_Vertical, symbol Device:Jumper
- removed R55, R56: 10k, Resistor_SMD:R_0805_2012Metric_Pad1.20x1.40mm_HandSolder, symbol Device:R
- removed R57, R58, R61, R66: 22k, Resistor_SMD:R_0805_2012Metric_Pad1.20x1.40mm_HandSolder, symbol Device:R
- removed R60: 4.7k, Resistor_SMD:R_0805_2012Metric_Pad1.20x1.40mm_HandSolder, symbol Device:R
- removed R62, R68: 1k, Resistor_SMD:R_0805_2012Metric_Pad1.20x1.40mm_HandSolder, symbol Device:R
- removed R63: 2.2k, Resistor_SMD:R_0805_2012Metric_Pad1.20x1.40mm_HandSolder, symbol Device:R
- removed R65: 240k, Resistor_SMD:R_0805_2012Metric_Pad1.20x1.40mm_HandSolder, symbol Device:R
- removed SW1: SW_DIP_x05, Button_Switch_THT:SW_DIP_SPSTx05_Slide_6.7x14.26mm_W7.62mm_P2.54mm_LowProfile, symbol Switch:SW_DIP_x05
- removed U15: 8580, Package_DIP:DIP-28_W15.24mm_Socket, symbol 65xx:8580
- removed U18: L78L09_SOT89, Package_TO_SOT_SMD:SOT-89-3, symbol Regulator_Linear:L78L09_SOT89
- removed U19: ATmega88PA-AU, Package_QFP:TQFP-32_7x7mm_P0.8mm, symbol MCU_Microchip_ATmega:ATmega88PA-AU
- R53: value 1k -> 10k
- R54: value 330k -> 10k
Connections:
- net BUS0 is gone; now on net A11: U7.6 (IO)
- net BUS1 is gone; now on net A10: U7.5 (IO)
- net GNDA is gone; now on net GND: C12.2, C15.2, C16.2, C17.2, C20.2, C23.2, C24.2, C25.2, C26.2, C27.2, C28.2, C29.2, C30.2, C31.2, C32.2, C33.2, C42.2, C43.2, C44.2, C45.2, C46.2, C47.2, C6.1, C60.1, C61.1, C62.1, C63.1, C64.1, C65.1, C66.1, C67.1, C68.2, C69.2, C70.2, C71.2, C77.2, C78.2, C83.2, C89.1, C90.2, C92.2, C96.2, C98.2, R10.1, R11.1, R12.1, R36.1, R37.1, R38.1, R9.2, U1.4 (V-), U10.6 (Vss), U11.10 (A0), U11.13 (GND), U11.14 (~{CS}), U11.15 (~{RD}), U11.18 (GND), U11.25 (GND), U11.36 (GND), U11.4 (AGND), U11.45 (GND), U11.48 (GND), U11.49 (GND), U11.7 (MICIN), U11.9 (GND), U14.9 (GND), U16.1 (GND), U17.1 (GND), U2.4 (V-), U20.1 (GND), U21.1 (GND), U23.10 (GND), U23.19 (CE), U4.1 (GND), U4.17 (AGND), U5.6 (Vss), U6.4 (V-), U9.1 (GND), U9.17 (AGND)
- net ~{BUSACK} is gone; now on net AD2: U7.93 (IO)
- net ~{BUSRQ} is gone; now on net AD4: U7.97 (IO)
- net ~{HALT} is gone; now on net AD3: U7.96 (IO)
- net ~{INT} is gone; now on net A5: U7.143 (IO)
- net ~{MREQ} is gone; now on net A3: U7.131 (IO)
- net ~{NMI} is gone; now on net A8: U7.1 (IO)
- net ~{RFSH} is gone; now on net D3: U7.122 (IO)
- net ~{ROMCSB} is gone; now on net A14: U7.106 (IO)
- net +5V: now also R53.1, R54.1
- net A0: now also U7.117 (IO); no longer U7.139 (IO)
- net A1: now also U7.119 (IO); no longer U7.138 (IO)
- net A10: no longer U7.103 (IO)
- net A11: no longer U7.102 (IO)
- net A12: now also U7.108 (IO); no longer U7.100 (IO)
- net A13: now also U7.109 (IO); no longer U7.116 (IO)
- net A14: no longer U7.120 (IO)
- net A15: now also U7.107 (IO); no longer U7.119 (IO)
- net A2: now also U7.121 (IO); no longer U7.137 (IO)
- net A3: no longer U7.136 (IO)
- net A4: now also U7.141 (IO); no longer U7.134 (IO)
- net A5: no longer U7.140 (IO)
- net A6: now also U7.140 (IO); no longer U7.133 (IO)
- net A7: now also U7.139 (IO); no longer U7.132 (IO)
- net A8: no longer U7.98 (IO)
- net A9: now also U7.2 (IO); no longer U7.101 (IO)
- net AA0: now also U7.88 (IO); no longer U7.23 (IO)
- net AD0: now also U7.91 (IO); no longer U7.27 (IO)
- net AD1: now also U7.92 (IO); no longer U7.7 (IO)
- net AD2: no longer U7.8 (IO)
- net AD3: no longer U7.9 (IO)
- net AD4: no longer U7.10 (IO)
- net AD5: now also U7.98 (IO); no longer U7.11 (IO)
- net AD6: now also U7.99 (IO); no longer U7.12 (IO)
- net AD7: now also U7.100 (IO); no longer U7.14 (IO)
- net CFG0: now also R49.2, SW2.1, U7.61 (IO); no longer R51.2, U7.90 (IO)
- net CFG1: now also SW2.2, U7.60 (IO); no longer U7.91 (IO)
- net CFG2: now also R51.2, SW2.3, U7.56 (IO); no longer R49.2, U7.92 (IO)
- net D0: now also U7.112 (IO); no longer U7.141 (IO)
- net D1: now also U7.113 (IO); no longer U7.142 (IO)
- net D2: now also U7.116 (IO); no longer U7.2 (IO)
- net D3: no longer U7.118 (IO)
- net D4: now also U7.132 (IO); no longer U7.117 (IO)
- net D5: now also U7.120 (IO); no longer U7.112 (IO)
- net D6: now also U7.118 (IO); no longer U7.110 (IO)
- net D7: now also U7.110 (IO); no longer U7.108 (IO)
- net FM1_ENA: now also U7.82 (IO); no longer U7.29 (IO)
- net FM2_ENA: now also U7.81 (IO); no longer U7.28 (IO)
- net GA0: now also U7.34 (IO); no longer U7.68 (IO)
- net GA1: now also U7.32 (IO); no longer U7.67 (IO)
- net GA10: now also U7.14 (IO); no longer U7.46 (IO)
- net GA11: now also U7.7 (IO); no longer U7.40 (IO)
- net GA12: now also U7.9 (IO); no longer U7.42 (IO)
- net GA13: now also U12.5 (A7), U22.5 (A7), U7.10 (IO); no longer U12.28 (A13), U22.28 (A13), U7.43 (IO)
- net GA14: now also U12.28 (A13), U22.28 (A13), U7.11 (IO); no longer U12.3 (A14), U22.3 (A14), U7.44 (IO)
- net GA15: now also U7.12 (IO); no longer U7.45 (IO)
- net GA2: now also U7.31 (IO); no longer U7.66 (IO)
- net GA3: now also U7.30 (IO); no longer U7.65 (IO)
- net GA4: now also U7.28 (IO); no longer U7.62 (IO)
- net GA5: now also U7.25 (IO); no longer U7.60 (IO)
- net GA6: now also U7.22 (IO); no longer U7.55 (IO)
- net GA7: now also U12.3 (A14), U22.3 (A14), U7.19 (IO); no longer U12.5 (A7), U22.5 (A7), U7.53 (IO)
- net GA8: now also U7.16 (IO); no longer U7.48 (IO)
- net GA9: now also U7.15 (IO); no longer U7.47 (IO)
- net GCLK: now also U7.8 (IO); no longer U7.41 (IO)
- net GD0: now also U12.17 (D3), U22.17 (D3), U7.37 (IO); no longer U12.13 (D0), U22.13 (D0), U7.71 (IO)
- net GD1: now also U12.15 (D2), U22.15 (D2), U7.40 (IO); no longer U12.14 (D1), U22.14 (D1), U7.75 (IO)
- net GD2: now also U12.18 (D4), U22.18 (D4), U7.42 (IO); no longer U12.15 (D2), U22.15 (D2), U7.79 (IO)
- net GD3: now also U12.14 (D1), U22.14 (D1), U7.43 (IO); no longer U12.17 (D3), U22.17 (D3), U7.80 (IO)
- net GD4: now also U12.19 (D5), U22.19 (D5), U7.44 (IO); no longer U12.18 (D4), U22.18 (D4), U7.81 (IO)
- net GD5: now also U12.13 (D0), U22.13 (D0), U7.41 (IO); no longer U12.19 (D5), U22.19 (D5), U7.78 (IO)
- net GD6: now also U7.39 (IO); no longer U7.74 (IO)
- net GD7: now also U7.38 (IO); no longer U7.72 (IO)
- net GDAC0: now also U23.9 (A7), U7.66 (IO); no longer R26.2, U23.3 (A1), U7.39 (IO)
- net GDAC1: now also U23.7 (A5), U7.65 (IO); no longer R32.2, U23.5 (A3), U7.38 (IO)
- net GDAC2: now also U23.5 (A3), U7.63 (IO); no longer R35.2, U23.7 (A5), U7.37 (IO)
- net GDAC3: now also U23.3 (A1), U7.62 (IO); no longer R39.2, U23.9 (A7), U7.36 (IO)
- net GMA15: now also U7.49 (IO); no longer U7.87 (IO)
- net GMA16: now also U7.35 (IO); no longer U7.69 (IO)
- net GMA17: now also U7.36 (IO); no longer U7.70 (IO)
- net GMA18: now also U7.48 (IO); no longer U7.86 (IO)
- net GND: now also SW2.10, SW2.6, SW2.7, SW2.8, SW2.9; no longer R53.2, R54.2
- net MIDI_CLK: now also U7.103 (IO); no longer U7.35 (IO)
- net SAA_CLK: now also U7.102 (IO); no longer U7.16 (IO)
- net YM_M: now also U7.90 (IO); no longer U7.25 (IO)
- net ~{ARD}: now also U7.87 (IO); no longer U7.22 (IO)
- net ~{AWR}: now also U7.86 (IO); no longer U7.21 (IO)
- net ~{DOS}: now also U7.111 (IO)
- net ~{GINT}: now also U7.18 (IO); no longer U7.49 (IO)
- net ~{GIORQ}: now also U7.23 (IO); no longer U7.56 (IO)
- net ~{GM1}: now also U7.29 (IO); no longer U7.63 (IO)
- net ~{GMREQ}: now also U7.21 (IO); no longer U7.54 (IO)
- net ~{GRAM}: now also U7.46 (IO); no longer U12.22 (~{CE}), U7.83 (IO)
- net ~{GRD}: now also U7.45 (IO); no longer U7.82 (IO)
- net ~{GRESET}: now also U7.27 (IO); no longer U7.61 (IO)
- net ~{GROM}: now also U7.53 (IO); no longer U7.88 (IO)
- net ~{GWR}: now also U7.47 (IO); no longer U7.84 (IO)
- net ~{IORQGE1}: now also U7.133 (IO); no longer U7.113 (IO)
- net ~{IORQ}: now also U7.134 (IO); no longer U7.107 (IO)
- net ~{M1}: now also U7.142 (IO); no longer U7.121 (IO)
- net ~{RD}: now also U7.136 (IO); no longer U7.111 (IO)
- net ~{RST}: now also U7.80 (IO); no longer U7.30 (IO)
- net ~{SAA_CS}: now also U7.101 (IO); no longer U7.15 (IO)
- net ~{WAIT}: now also U7.138 (IO); no longer U7.99 (IO)
- net ~{WR}: now also U7.137 (IO); no longer U7.109 (IO)
- net ~{YM1_CS}: now also U7.83 (IO); no longer U7.18 (IO)
- net ~{YM2_CS}: now also U7.84 (IO); no longer U7.19 (IO)
- net CFG3: now reaches SW2.4
- net CFG3: now also R54.2, U7.55 (IO)
- net CFG4: now reaches SW2.5
- net CFG4: now also R53.2, U7.54 (IO)
- net at U23.11 (B7): now also R26.2
- net at U23.13 (B5): now also R32.2
- net at U23.15 (B3): now also R35.2
- net at U23.17 (B1): now also R39.2
- net CLKCPU: no longer names the net of U7.125 (IN/GCLK1)
- new net ~{GRAM1}: U12.22 (~{CE})
- no-connect marks 76 -> 70
Other:
- note removed: "+12V for 6581 +9V for 8580"
- note removed: "470p for 6581 22n for 8580"
- note removed: "For 256K RAM compatibility: GMA18<->A17 GMA17<->A18"
- moved on the sheet: C1, C10, C11, C12, C13, C14, C15, C16, C17, C18, C19, C2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

Commit message: wip pcb rev.A
Connections:
- net +5VA: no longer R42.2, R43.2, R48.2
- net +5VA_2: now also R42.2, R43.2, R48.2
- net AA0: now also U7.83 (IO); no longer U7.88 (IO)
- net FM1_ENA: now also U7.80 (IO); no longer U7.82 (IO)
- net FM2_ENA: now also U7.90 (IO); no longer U7.81 (IO)
- net GDAC0: now also U23.8 (A6); no longer U23.9 (A7)
- net GDAC1: now also U23.6 (A4); no longer U23.7 (A5)
- net GDAC2: now also U23.4 (A2); no longer U23.5 (A3)
- net GDAC3: now also U23.2 (A0); no longer U23.3 (A1)
- net YM_M: now also U7.82 (IO); no longer U7.90 (IO)
- net ~{ARD}: now also U7.84 (IO); no longer U7.87 (IO)
- net ~{RST}: now also U7.88 (IO); no longer U7.80 (IO)
- net ~{YM1_CS}: now also U7.81 (IO); no longer U7.83 (IO)
- net ~{YM2_CS}: now also U7.87 (IO); no longer U7.84 (IO)
- net at R32.2: now also U23.14 (B4); no longer U23.13 (B5)
- net at R26.2: now also U23.12 (B6); no longer U23.11 (B7)
- net at R39.2: now also U23.18 (B0); no longer U23.17 (B1)
- net at R35.2: now also U23.16 (B2); no longer U23.15 (B3)

Commit message: wip pcb rev.A
Parts:
- added J5: Conn_01x04, Connector_PinHeader_2.54mm:PinHeader_1x04_P2.54mm_Vertical, symbol Connector_Generic:Conn_01x04
- added R55, R56: 24k, Resistor_SMD:R_0805_2012Metric_Pad1.20x1.40mm_HandSolder, symbol Device:R
Connections:
- net ~{GRAM} is gone; now on net ~{GROM}: U7.46 (IO)
- net +3V3: now also R49.1, R50.1, R51.1, R53.1, R54.1
- net +5V: no longer R49.1, R50.1, R51.1, R53.1, R54.1
- net +5VA_1: now also C90.1, U20.2 (VO); no longer C78.1, U17.2 (VO)
- net +5VA_2: now also C78.1, U17.2 (VO); no longer C90.1, U20.2 (VO)
- net A0: now also U7.111 (IO); no longer U7.117 (IO)
- net A1: now also U7.113 (IO); no longer U7.119 (IO)
- net A10: now also U7.141 (IO); no longer U7.5 (IO)
- net A11: now also U7.142 (IO); no longer U7.6 (IO)
- net A12: now also U7.102 (IO); no longer U7.108 (IO)
- net A13: now also U7.103 (IO); no longer U7.109 (IO)
- net A14: now also U7.100 (IO); no longer U7.106 (IO)
- net A15: now also U7.101 (IO); no longer U7.107 (IO)
- net A2: now also U7.117 (IO); no longer U7.121 (IO)
- net A3: now also U7.119 (IO); no longer U7.131 (IO)
- net A4: now also U7.138 (IO); no longer U7.141 (IO)
- net A5: now also U7.136 (IO); no longer U7.143 (IO)
- net A6: now also U7.134 (IO); no longer U7.140 (IO)
- net A7: now also U7.133 (IO); no longer U7.139 (IO)
- net A8: now also U7.139 (IO); no longer U7.1 (IO)
- net A9: now also U7.140 (IO); no longer U7.2 (IO)
- net AA0: now also U7.78 (IO); no longer U7.83 (IO)
- net AD0: now also U7.86 (IO); no longer U7.91 (IO)
- net AD1: now also U7.87 (IO); no longer U7.92 (IO)
- net AD2: now also U7.88 (IO); no longer U7.93 (IO)
- net AD3: now also U7.90 (IO); no longer U7.96 (IO)
- net AD4: now also U7.91 (IO); no longer U7.97 (IO)
- net AD5: now also U7.92 (IO); no longer U7.98 (IO)
- net AD6: now also U7.93 (IO); no longer U7.99 (IO)
- net AD7: now also U7.96 (IO); no longer U7.100 (IO)
- net CFG0: now also U7.48 (IO); no longer U7.61 (IO)
- net CFG1: now also U7.49 (IO); no longer U7.60 (IO)
- net CFG2: now also U7.53 (IO); no longer U7.56 (IO)
- net CFG3: now also U7.54 (IO); no longer U7.55 (IO)
- net CFG4: now also U7.55 (IO); no longer U7.54 (IO)
- net D0: now also U7.108 (IO); no longer U7.112 (IO)
- net D1: now also U7.109 (IO); no longer U7.113 (IO)
- net D2: now also U7.110 (IO); no longer U7.116 (IO)
- net D3: now also U7.118 (IO); no longer U7.122 (IO)
- net D4: now also U7.120 (IO); no longer U7.132 (IO)
- net D5: now also U7.116 (IO); no longer U7.120 (IO)
- net D6: now also U7.112 (IO); no longer U7.118 (IO)
- net D7: now also U7.106 (IO); no longer U7.110 (IO)
- net FM1_ENA: now also U7.74 (IO); no longer U7.80 (IO)
- net FM2_ENA: now also U7.84 (IO); no longer U7.90 (IO)
- net GA0: now also U7.10 (IO); no longer U7.34 (IO)
- net GA1: now also U7.11 (IO); no longer U7.32 (IO)
- net GA10: now also U7.23 (IO); no longer U7.14 (IO)
- net GA11: now also U7.30 (IO); no longer U7.7 (IO)
- net GA12: now also U7.31 (IO); no longer U7.9 (IO)
- net GA13: now also U7.32 (IO); no longer U7.10 (IO)
- net GA14: now also U7.34 (IO); no longer U7.11 (IO)
- net GA15: now also U7.35 (IO); no longer U7.12 (IO)
- net GA2: now also U7.12 (IO); no longer U7.31 (IO)
- net GA3: now also U7.14 (IO); no longer U7.30 (IO)
- net GA4: now also U7.15 (IO); no longer U7.28 (IO)
- net GA5: now also U7.16 (IO); no longer U7.25 (IO)
- net GA6: now also U7.18 (IO); no longer U7.22 (IO)
- net GA8: now also U7.21 (IO); no longer U7.16 (IO)
- net GA9: now also U7.22 (IO); no longer U7.15 (IO)
- net GCLK: now also U7.41 (IO); no longer U7.8 (IO)
- net GD0: now also U7.44 (IO); no longer U7.37 (IO)
- net GD1: now also U7.45 (IO); no longer U7.40 (IO)
- net GD3: now also U7.37 (IO); no longer U7.43 (IO)
- net GD4: now also U7.40 (IO); no longer U7.44 (IO)
- net GD5: now also U7.38 (IO); no longer U7.41 (IO)
- net GD7: now also U7.43 (IO); no longer U7.38 (IO)
- net GDAC0: now also U7.63 (IO); no longer U7.66 (IO)
- net GDAC1: now also U7.62 (IO); no longer U7.65 (IO)
- net GDAC2: now also U7.61 (IO); no longer U7.63 (IO)
- net GDAC3: now also U7.60 (IO); no longer U7.62 (IO)
- net GMA15: now also U7.47 (IO); no longer U7.49 (IO)
- net GMA16: now also U7.2 (IO); no longer U7.35 (IO)
- net GMA17: now also U7.5 (IO); no longer U7.36 (IO)
- net GMA18: now also U7.6 (IO); no longer U7.48 (IO)
- net GND: now also J5.2 (Pin_2), J5.3 (Pin_3)
- net MIDI_CLK: now also U7.99 (IO); no longer U7.103 (IO)
- net SAA_CLK: now also U7.98 (IO); no longer U7.102 (IO)
- net YM_M: now also U7.75 (IO); no longer U7.82 (IO)
- net ~{ARD}: now also U7.79 (IO); no longer U7.84 (IO)
- net ~{AWR}: now also U7.80 (IO); no longer U7.86 (IO)
- net ~{DOS}: now also U7.107 (IO); no longer U7.111 (IO)
- net ~{GINT}: now also U7.36 (IO); no longer U7.18 (IO)
- net ~{GIORQ}: now also U7.28 (IO); no longer U7.23 (IO)
- net ~{GM1}: now also U7.8 (IO); no longer U7.29 (IO)
- net ~{GMREQ}: now also U7.29 (IO); no longer U7.21 (IO)
- net ~{GRAM1}: now also U7.7 (IO)
- net ~{GRAM2}: now also U7.1 (IO)
- net ~{GRD}: now also U7.27 (IO); no longer U7.45 (IO)
- net ~{GRESET}: now also U7.9 (IO); no longer U7.27 (IO)
- net ~{GROM}: no longer U7.53 (IO)
- net ~{GWR}: now also U7.25 (IO); no longer U7.47 (IO)
- net ~{IORQGE1}: now also U7.121 (IO); no longer U7.133 (IO)
- net ~{IORQ}: now also U7.122 (IO); no longer U7.134 (IO)
- net ~{M1}: now also U7.137 (IO); no longer U7.142 (IO)
- net ~{RD}: now also U7.126 (IN/OE1); no longer U7.136 (IO)
- net ~{RST}: now also U7.83 (IO); no longer U7.88 (IO)
- net ~{SAA_CS}: now also U7.97 (IO); no longer U7.101 (IO)
- net ~{WAIT}: now also U7.132 (IO); no longer U7.138 (IO)
- net ~{WR}: now also U7.131 (IO); no longer U7.137 (IO)
- net ~{YM2_CS}: now also U7.82 (IO); no longer U7.87 (IO)
- net at R1.1, R13.1, R14.1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: now also R55.1
- net at R19.1, R21.1, R22.1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: now also R56.1
- net MIX_L renamed SND_L
- net MIX_R renamed SND_R
- new net IN_L: J5.4 (Pin_4), R55.2
- new net IN_R: J5.1 (Pin_1), R56.2
Other:
- moved on the sheet: C1, C10, C11, C13, C14, C18, C19, C2, C21, C22, C26, C27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

Commit message: wip pcb rev.A
Parts:
- added C37: 100n, Capacitor_SMD:C_0805_2012Metric_Pad1.18x1.45mm_HandSolder, symbol Device:C
- added R57, R58: 10k, Resistor_SMD:R_0805_2012Metric_Pad1.20x1.40mm_HandSolder, symbol Device:R
- added R59: 24k, Resistor_SMD:R_0805_2012Metric_Pad1.20x1.40mm_HandSolder, symbol Device:R
- added TP1: TestPoint, TestPoint:TestPoint_Pad_D1.0mm, symbol Connector:TestPoint
- added X2: ??MHz, Oscillator:Oscillator_SMD_SeikoEpson_SG8002CA-4Pin_7.0x5.0mm, symbol Oscillator:XO91
- H1, H2: now left out of the parts list
Connections:
- net +3V3: now also C88.2, X1.1 (EN), X1.4 (V+), C37.2, R57.1, R58.1, R59.1, X2.1 (EN), X2.4 (V+)
- net +5V: no longer C88.2, X1.1 (EN), X1.4 (V+)
- net A10: now also U7.142 (IO); no longer U7.141 (IO)
- net A11: now also U7.143 (IO); no longer U7.142 (IO)
- net A4: now also U7.139 (IO); no longer U7.138 (IO)
- net A5: now also U7.137 (IO); no longer U7.136 (IO)
- net A6: now also U7.136 (IO); no longer U7.134 (IO)
- net A7: now also U7.134 (IO); no longer U7.133 (IO)
- net A8: now also U7.140 (IO); no longer U7.139 (IO)
- net A9: now also U7.141 (IO); no longer U7.140 (IO)
- net GMA16: now also U7.5 (IO); no longer U7.2 (IO)
- net GMA17: now also U7.2 (IO); no longer U7.5 (IO)
- net GND: now also H1.1, H2.1, C37.1, X2.2 (GND)
- net ~{DOS}: now also R57.2
- net ~{M1}: now also U7.138 (IO); no longer U7.137 (IO)
- net ~{RD}: now also R59.2
- net ~{WAIT}: now also U7.133 (IO); no longer U7.132 (IO)
- net CLKx: now reaches U7.125 (IN/GCLK1)
- net CLKx: now also X2.3 (OUT)
- net at U7.72 (IO): now also TP1.1
- net ~{IODOS}: now reaches J4.b20 (Pin_b20)
- net ~{IODOS}: now also U7.132 (IO), R58.2
- net ~{IORQGE1} renamed ~{IORQGE}
- no-connect marks 70 -> 72
Other:
- moved on the sheet: C38, C39, C40, C87, C88, J4
