File: pcb/rev.A/zx-multisound.kicad_pcb (KiCad board)
At the start: 2 copper layers, 170 x 63.6 mm, 177 parts, among them J1 PJ307, J2 Conn_01x04, J3 Conn_01x04, J4 Conn_02x31_Row_Letter_First, J5 PinHeader, SW1 SW_DIP_x05, U1 MCP602, U10 YM2203, U11 27C512, U12 YM3014B, U13 SAM2695, U14 74ACT245, U15 AMS1117-3.3, U16 NCP1117-5.0_TO252, U17 NCP1117-5.0_TO252, U18 NCP1117-5.0_TO252, U19 AMS1117-3.3, U2 MCP602, U20 SAA1099, U3 AS6C4008-55SIN, U4 YM2203, U5 Z84C0020PEC, U6 YM3014B, U7 MCP602, U8 EPM3256ATC144, U9 AS6C4008-55SIN, X1 32MHz, X2 ??MHz

Commit message: wip pcb rev.A
Parts:
- C42: footprint Capacitor_SMD:C_1206_3216Metric_Pad1.33x1.80mm_HandSolder -> Capacitor_Tantalum_SMD:CP_EIA-3216-18_Kemet-A_Pad1.58x1.35mm_HandSolder
- moved C42 0.20 mm to (63.1, 118.2)

Commit message: wip pcb rev.A
Parts:
- C30, C31, C32, C47: value 1n -> 10n
- C34: footprint Capacitor_SMD:C_1206_3216Metric_Pad1.33x1.80mm_HandSolder -> Capacitor_Tantalum_SMD:CP_EIA-3216-18_Kemet-A_Pad1.58x1.35mm_HandSolder
- R12, R30, R31, R6: value 24k -> 33k
- R2, R33: value 24k -> 18k
- R43, R44, R45, R50: value 2.2k -> 1k
- U15, U19: value AMS1117-3.3 -> 1117-3.3
- U16, U17, U18: value NCP1117-5.0_TO252 -> 78M05
- U5: value Z84C0020PEC -> Z84C0020FEC
- moved C37 6.98 mm to (77.6, 77.8), turned to 180 degrees
- moved C35 6.15 mm to (62.8, 87.8)
- moved C34 3.86 mm to (191.0, 114.0)
- moved C39 3.27 mm to (183.7, 75.8), turned to -90 degrees
- moved R53 1.05 mm to (196.2, 88.7)
- moved R54 1.05 mm to (191.2, 77.2)
- moved R56 1.05 mm to (196.2, 77.2)
- moved R57 1.05 mm to (198.8, 77.2)
- moved R59 1.05 mm to (192.3, 88.7)
- moved J5 1.05 mm to (191.2, 86.6)
- moved R52 1.05 mm to (200.1, 88.7)
- moved R55 1.05 mm to (193.7, 77.2)
- moved R58 1.05 mm to (201.3, 77.2)
- moved SW1 1.05 mm to (191.2, 81.0)
- moved U16 0.78 mm to (62.9, 84.5), turned to 90 degrees
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Connections:
- H1 pad 1: GND -> unconnected-(H1-Pad1)
- H2 pad 1: GND -> unconnected-(H2-Pad1)
- U16 pad 1: GND -> +12V
- U16 pad 2: +5VA -> GND
- U16 pad 3: +12V -> +5VA
- U17 pad 1: GND -> +12V
- U17 pad 2: +5VA_2 -> GND
- U17 pad 3: +12V -> +5VA_2
- U18 pad 1: GND -> +12V
- U18 pad 2: +5VA_1 -> GND
- U18 pad 3: +12V -> +5VA_1
Routing:
- net +12V: track 335.8 -> 345.1 mm, vias 6 -> 9
- net GND: track 231.7 -> 240.6 mm, vias 251 -> 329
- net +5VA: track 109.0 -> 101.5 mm, vias 33 -> 5
- net +5VA_1: track 100.5 -> 107.2 mm, vias 34 -> 4
- net +5VA_2: track 113.3 -> 115.3 mm, vias 35 -> 5
- net /TCK: track 50.7 -> 48.9 mm
- net /TDI: track 43.7 -> 41.9 mm
- net +3V3: track 210.9 -> 209.3 mm
- net /TMS: track 27.3 -> 26.2 mm
- net +5V: track 307.1 -> 308.2 mm
- net /~{GROM}: track 48.1 -> 49.1 mm
- net /GMA15: track 105.0 -> 105.9 mm
- removed copper zone on B.Cu, net +5VA
- removed copper zone on B.Cu, net +5VA_1
- removed copper zone on B.Cu, net +5VA_2

Commit message: wip pcb rev.A
Parts:
- added C84: 100n, Capacitor_SMD:C_0805_2012Metric_Pad1.18x1.45mm_HandSolder, B.Cu at (161.6, 122.4)
- added REF**: NPTH_D=0.4mm, my:NPTH_D=0.4mm, F.Cu at (184.7, 127.6)
- added REF**1: NPTH_D=0.4mm, my:NPTH_D=0.4mm, F.Cu at (184.7, 128.6)
- added REF**2: NPTH_D=0.4mm, my:NPTH_D=0.4mm, F.Cu at (184.7, 129.6)
- added REF**3: NPTH_D=0.4mm, my:NPTH_D=0.4mm, F.Cu at (184.7, 130.6)
- added REF**4: NPTH_D=0.4mm, my:NPTH_D=0.4mm, F.Cu at (184.7, 131.6)
- added REF**5: NPTH_D=0.4mm, my:NPTH_D=0.4mm, F.Cu at (184.7, 132.6)
- added REF**6: NPTH_D=0.4mm, my:NPTH_D=0.4mm, F.Cu at (184.7, 133.5)
- added REF**7: NPTH_D=0.4mm, my:NPTH_D=0.4mm, F.Cu at (184.7, 134.5)
- added REF**8: NPTH_D=0.4mm, my:NPTH_D=0.4mm, F.Cu at (185.6, 127.6)
- added REF**9: NPTH_D=0.4mm, my:NPTH_D=0.4mm, F.Cu at (186.6, 127.6)
- added U21: 74LVC1G125DB, Package_TO_SOT_SMD:SOT-23-5_HandSoldering, B.Cu at (164.6, 122.4)
- C34, C42: value 10u -> 22u
- C36, C38, C40: value 47u/16V -> 100u/10V
- J4: footprint my:ZX_NEMO_EDGE -> my:ZX_NEMO_60_EDGE
- U1, U2, U7: value MCP602 -> LM358D
- moved H1 0.08 mm to (61.6, 124.6)
- moved H2 0.07 mm to (61.6, 74.6)
Connections:
- net +3V3 renamed +3.3V
- J4 pad a13: ~{IORQGE} -> Net-(J4-Pada13)
Routing:
- net Net-(J4-Pada13): track 0.00 -> 33.8 mm, vias 0 -> 2
- net ~{IORQGE}: track 40.8 -> 12.0 mm
- net +5V: track 308.2 -> 317.6 mm
- net /TDI: track 41.9 -> 46.3 mm
- net ~{IORQ}: track 31.4 -> 32.1 mm
Other:
- outline, holes or cut-outs redrawn
