File: pcb/rev.A/zx-multisound.kicad_sch (KiCad schematic)
At the start: 172 parts, among them J1 PJ307, J2 PinHeader, J3 Conn_01x04, J4 Conn_02x31_Row_Letter_First, J5 Conn_01x04, SW2 SW_DIP_x05, U1 MCP602, U10 YM3014B, U11 SAM2695, U12 AS6C4008-55SIN, U13 AMS1117-3.3, U14 SAA1099, U16 AMS1117-3.3, U17 NCP1117-5.0_TO252, U2 MCP602, U20 NCP1117-5.0_TO252, U21 NCP1117-5.0_TO252, U22 AS6C4008-55SIN, U23 74HC245, U3 Z84C0020PEC, U4 YM2203, U5 YM3014B, U6 MCP602, U7 EPM3256ATC144, U8 27C512, U9 YM2203, X1 32MHz, X2 ??MHz

Commit message: wip pcb rev.A
Parts:
- removed R20: 2.2k, Resistor_SMD:R_0805_2012Metric_Pad1.20x1.40mm_HandSolder, symbol Device:R
- added C82, C83: 10u, Capacitor_SMD:CP_Elec_4x5.4, symbol Device:C_Polarized
- added R19: 47k, Resistor_SMD:R_0805_2012Metric_Pad1.20x1.40mm_HandSolder, symbol Device:R
- added TP2, TP3, TP4: TestPoint, TestPoint:TestPoint_Pad_D1.0mm, symbol Connector:TestPoint
- C1, C10, C11, C2, C3, C7, C8, C9: symbol Device:CP -> Device:C_Polarized
- C12: renamed from C13; symbol Device:CP -> Device:C_Polarized
- C13: renamed from C15; symbol Device:CP -> Device:C_Polarized
- C14: renamed from C16; symbol Device:CP -> Device:C_Polarized
- C16: renamed from C14; symbol Device:CP -> Device:C_Polarized
- C17: renamed from C18; symbol Device:CP -> Device:C_Polarized
- C18: renamed from C19; symbol Device:CP -> Device:C_Polarized
- C19: renamed from C21; symbol Device:CP -> Device:C_Polarized
- C21: renamed from C22; symbol Device:CP -> Device:C_Polarized
- C22: renamed from C28; symbol Device:CP -> Device:C_Polarized
- C23: renamed from C29; symbol Device:CP -> Device:C_Polarized
- C36: renamed from C77; symbol Device:CP -> Device:C_Polarized
- C38: renamed from C78; symbol Device:CP -> Device:C_Polarized
- C40: renamed from C90; symbol Device:CP -> Device:C_Polarized
- C5: renamed from C4; symbol Device:CP -> Device:C_Polarized
- C6: renamed from C5; symbol Device:CP -> Device:C_Polarized
- C75: renamed from C34; symbol Device:CP -> Device:C_Polarized
- C76: renamed from C84; symbol Device:CP -> Device:C_Polarized
- LOGO1: footprint mygraphic:black-mage-9.6x6.5 -> mygraphic:black-mage-12.5x8.6
- R15, R25: value 24k -> 10K
- R7: value 2.2k -> 47k
- U14: renamed from U23; value 74HC245 -> 74ACT245
- renumbered C17 to C15, C23 to C20, C30 to C24, C26 to C25, C27 to C26, C31 to C27, C32 to C28, C33 to C29, C25 to C30, C24 to C31, C20 to C32, C35 to C33, C36 to C34, C92 to C35, C96 to C37, C98 to C39, C6 to C4, C42 to C41, C83 to C42, C44 to C43, C45 to C44, C46 to C45, C47 to C46, C12 to C47, C88 to C60, C37 to C61, C38 to C62, C39 to C63, C40 to C64, C87 to C65, C65 to C66, C66 to C67, C67 to C68, C60 to C69, C62 to C70, C89 to C71, C64 to C72, C61 to C73, C63 to C74, C68 to C77, C69 to C78, C70 to C79, C71 to C80, C43 to C81, J3 to J2, J5 to J3, J2 to J5, R55 to R1, R12 to R10, R9 to R11, R6 to R12, R8 to R13, R13 to R14, R14 to R16, R16 to R17, R17 to R18, R1 to R2, R18 to R20, R19 to R21, R23 to R22, R24 to R23, R21 to R24, R22 to R26, R33 to R32, R34 to R33, R56 to R34, R36 to R35, R37 to R36, R38 to R37, R58 to R38, R40 to R39, R2 to R4, R41 to R40, R57 to R41, R59 to R42, R39 to R43, R35 to R44, R32 to R45, R42 to R46, R43 to R47, R44 to R48, R45 to R49, R26 to R50, R48 to R51, R46 to R52, R47 to R53, R49 to R54, R50 to R55, R51 to R56, R54 to R57, R53 to R58, R52 to R59, R4 to R6, R10 to R8, R11 to R9, SW2 to SW1, U2 to U1, U9 to U10, U8 to U11, U10 to U12, U11 to U13, U13 to U15, U21 to U16, U20 to U18, U16 to U19, U6 to U2, U14 to U20, U12 to U3, U3 to U5, U5 to U6, U1 to U7, U6 to U7, U7 to U8, U22 to U9
Connections:
- net +3V3: no longer R54.1, R55.1, R56.1, R57.1, R58.1
- net +5V: now also R54.1, R55.1, R56.1, R57.1, R58.1
- net GND: now also R7.2, U14.3 (A1), U14.5 (A3), U14.7 (A5), U14.9 (A7), R19.2
- net IN_L: now also R7.1
- net IN_R: now also R19.1
- net SND_L: now also C82.2; no longer R7.1
- net SND_R: now also C83.2
- net at R15.2, U1.1: now also C82.1; no longer R7.2
- net at R25.2, U1.7: now also C83.1
- net at U8.69 (IO): now also TP4.1
- net at U8.70 (IO): now also TP3.1
- net at U8.71 (IO): now also TP2.1
- no-connect marks 72 -> 81
Other:
- title: ZX-SIZIF-512-EXT -> ZX-MULTISOUND
- moved on the sheet: H1, H2, J3

Commit message: wip pcb rev.A
Parts:
- removed C42: 10u, Capacitor_SMD:C_1206_3216Metric_Pad1.33x1.80mm_HandSolder, symbol Device:C
- added C42: 10u, Capacitor_Tantalum_SMD:CP_EIA-3216-18_Kemet-A_Pad1.58x1.35mm_HandSolder, symbol Device:CP
Connections:
- net +3.3VA: now also C42.1
- net GND: now also C42.2
Changed lines of the file:
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@@
   (junction (at 271.78 247.015) (diameter 1.016) (color 0 0 0 0)
   )
-  (junction (at 481.965 229.87) (diameter 0) (color 0 0 0 0)
-  )
   (junction (at 320.675 256.54) (diameter 1.016) (color 0 0 0 0)
   )
@@
   (junction (at 309.245 149.225) (diameter 1.016) (color 0 0 0 0)
   )
+  (junction (at 481.965 229.87) (diameter 0) (color 0 0 0 0)
+  )
   (junction (at 346.075 266.7) (diameter 1.016) (color 0 0 0 0)
   )
@@
     (pin "2")
   )
+  (symbol (lib_id "Device:CP") (at 481.965 233.68 0) (unit 1)
+    (in_bom yes) (on_board yes)
+    (property "Reference" "C42" (id 0) (at 483.87 231.775 0)
+      (effects (font (size 0.9906 0.9906)))
+    )
+    (property "Value" "10u" (id 1) (at 483.87 235.585 0)
+      (effects (font (size 0.9906 0.9906)))
+    )
+    (property "Footprint" "Capacitor_Tantalum_SMD:CP_EIA-3216-18_Kemet-A_Pad1.58x1.35mm_HandSolder" (id 2) (at 482.9302 237.49 0)
+      (effects (font (size 1.27 1.27)) hide)
+    )
+    (property "Datasheet" "~" (id 3) (at 481.965 233.68 0)
+      (effects (font (size 1.27 1.27)) hide)
+    )
+    (pin "1")
+    (pin "2")
+  )
   (symbol (lib_id "power:GND") (at 321.945 274.32 0) (unit 1)
     (in_bom yes) (on_board yes)
@@
     (pin "1")
   )
-  (symbol (lib_id "Device:C") (at 481.965 233.68 0) (unit 1)
-    (in_bom yes) (on_board yes)
-    (property "Reference" "C42" (id 0) (at 485.775 231.775 0)
-      (effects (font (size 0.9906 0.9906)) (justify right))
-    )
-    (property "Value" "10u" (id 1) (at 485.775 235.585 0)
-      (effects (font (size 0.9906 0.9906)) (justify right))
-    )
-    (property "Footprint" "Capacitor_SMD:C_1206_3216Metric_Pad1.33x1.80mm_HandSolder" (id 2) (at 482.9302 237.49 0)
-      (effects (font (size 1.27 1.27)) hide)
-    )
-    (property "Datasheet" "~" (id 3) (at 481.965 233.68 0)
-      (effects (font (size 1.27 1.27)) hide)
-    )
-    (pin "1")
-    (pin "2")
-  )
   (symbol (lib_id "power:+3.3V") (at 497.205 154.94 0) (unit 1)
     (in_bom yes) (on_board yes)
@@
       (reference "C41") (unit 1) (value "10u") (footprint "Capacitor_SMD:C_1206_3216Metric_Pad1.33x1.80mm_HandSolder")
     )
-    (path "/84f1a6bb-83fa-4913-8004-29061790a042"
-      (reference "C42") (unit 1) (value "10u") (footprint "Capacitor_SMD:C_1206_3216Metric_Pad1.33x1.80mm_HandSolder")
+    (path "/4535f211-2852-408d-baa6-f62ce1ac9854"
+      (reference "C42") (unit 1) (value "10u") (footprint "Capacitor_Tantalum_SMD:CP_EIA-3216-18_Kemet-A_Pad1.58x1.35mm_HandSolder")
     )
     (path "/00000000-0000-0000-0000-000069eb9506"

Commit message: wip pcb rev.A
Parts:
- removed C34: 10u, Capacitor_SMD:C_1206_3216Metric_Pad1.33x1.80mm_HandSolder, symbol Device:C
- removed U16, U17, U18: NCP1117-5.0_TO252, Package_TO_SOT_SMD:TO-252-2, symbol Regulator_Linear:NCP1117-5.0_TO252
- added C34: 10u, Capacitor_Tantalum_SMD:CP_EIA-3216-18_Kemet-A_Pad1.58x1.35mm_HandSolder, symbol Device:CP
- added U16, U17, U18: 78M05, Package_TO_SOT_SMD:TO-252-2, symbol Regulator_Linear:LM78M05_TO252
- C30, C31, C32, C47: value 1n -> 10n
- R12, R30, R31, R6: value 24k -> 33k
- R2, R33: value 24k -> 18k
- R43, R44, R45, R50: value 2.2k -> 1k
- U15, U19: value AMS1117-3.3 -> 1117-3.3
- U5: value Z84C0020PEC -> Z84C0020FEC
Connections:
- net +12V: now also U16.1 (VI), U17.1 (VI), U18.1 (VI)
- net +3V3: now also C34.1
- net +5VA: now also U16.3 (VO)
- net +5VA_1: now also U18.3 (VO)
- net +5VA_2: now also U17.3 (VO)
- net GND: now also C34.2, U16.2 (GND), U17.2 (GND), U18.2 (GND); no longer H1.1, H2.1
- no-connect marks 81 -> 83

Commit message: wip pcb rev.A
Parts:
- added C84: 100n, Capacitor_SMD:C_0805_2012Metric_Pad1.18x1.45mm_HandSolder, symbol Device:C
- added U21: 74LVC1G125DB, Package_TO_SOT_SMD:SOT-23-5_HandSoldering, symbol 74xGxx:74LVC1G125
- C34, C42: value 10u -> 22u; symbol Device:CP -> Device:C_Polarized
- C36, C38, C40: value 47u/16V -> 100u/10V
- J4: footprint my:ZX_NEMO_EDGE -> my:ZX_NEMO_60_EDGE; symbol Connector_Generic:Conn_02x31_Row_Letter_First -> Connector_Generic:Conn_02x30_Row_Letter_First; now in the parts list
- U1: renamed from U7; value MCP602 -> LM358D
- U1, U2, U7: value MCP602 -> LM358D
- U2: renamed from U1; value MCP602 -> LM358D
- U7: renamed from U2; value MCP602 -> LM358D
Connections:
- net +5V: now also C84.2, U21.2, U21.5 (VCC)
- net GND: now also C84.1, U21.3 (GND)
- net ~{IORQGE}: now also U21.1; no longer J4.a13 (Pin_a13)
- net +3V3 renamed +3.3V
- new net: J4.a13 (Pin_a13), U21.4
- no-connect marks 83 -> 81
Other:
- moved on the sheet: C62, C63, C64, C65

Commit message: update pcb rev.A - final version; add errata
Parts:
- J4: now left out of the parts list
Changed lines of the file:
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@@
     (pin "8")
   )
-  (symbol (lib_id "my:YM3014B") (at 287.655 153.035 0) (unit 1)
+  (symbol (lib_name "YM3014B_1") (lib_id "my:YM3014B") (at 287.655 153.035 0) (unit 1)
     (in_bom yes) (on_board yes)
     (property "Reference" "U12" (id 0) (at 279.4 142.875 0)
@@
     (pin "1")
   )
-  (symbol (lib_id "my:YM2203") (at 249.555 64.77 0) (unit 1)
+  (symbol (lib_name "YM2203_1") (lib_id "my:YM2203") (at 249.555 64.77 0) (unit 1)
     (in_bom yes) (on_board yes)
     (property "Reference" "U4" (id 0) (at 239.395 29.21 0)
@@
   )
   (symbol (lib_id "Connector_Generic:Conn_02x30_Row_Letter_First") (at 473.075 168.275 0) (unit 1)
-    (in_bom yes) (on_board yes)
+    (in_bom no) (on_board yes)
     (property "Reference" "J4" (id 0) (at 474.345 128.905 0)
       (effects (font (size 1 1)))
